File: BlackMagicProbe.kicad_sch (KiCad schematic)
At the start: 73 parts, among them J2 JST, J3 MALE, J4 FEMALE, J8 BMDU, Q2 BC847, Q3 BC847, Q4 BC847, SW1 BMP_BOOT, SW1 BMP_DFU, U1 STM32F103CBTx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

Commit message: Consolidate BOM
Parts:
- D1: value PWR -> ORANGE
- D1: value GDB -> GREEN
- D1: value TPWR -> BLUE
- D1: value UART -> YELLOW
- D1: value ERR -> RED
- R13: footprint Capacitor_SMD:C_0805_2012Metric_Pad1.18x1.45mm_HandSolder -> Resistor_SMD:R_0805_2012Metric_Pad1.20x1.40mm_HandSolder
- R13: value 5K -> 5.1K
- SW1: value BMP_BOOT -> BUTTON
- SW1: value BMP_DFU -> BUTTON
Other:
- note added: "BOOT"
- note added: "DFU"
