File: Main_USB_HUB.kicad_sch (KiCad schematic)
At the start: 43 parts, among them IC1 GL850G-HH, J16 USB_C_Receptacle_USB2.0, J17 EXTPWR, Q5 DMP2305U-7, U28 M24C02-FMN, U29 LM2596S-5, U6 SRV05-4, Y1 12MHz

Commit message: Consolidate BOM
Parts:
- D1: value HUB_OK -> ORANGE
- D1: value EXT_PWR -> ORANGE
- R13: value 2.2K -> 2K
