File: PicoProbe.kicad_sch (KiCad schematic)
At the start: 42 parts, among them J2 JST, J3 MALE, J4 FEMALE, J7 UART, J9 SWD, SW1 PP_BOOT, U12 LP5907MFX-3.3, U2 W25Q128JVS, U3 RP2040, U6 SRV05-4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

Commit message: Consolidate BOM
Parts:
- D1: value T RUN -> GREEN
- D1: value PWR -> ORANGE
- D1: value UART RX -> BLUE
- D1: value UART TX -> BLUE
- D1: value DAP CONN -> YELLOW
- J7: value UART -> JST
- J9: value SWD -> JST
- R1, R5: footprint Capacitor_SMD:C_0805_2012Metric_Pad1.18x1.45mm_HandSolder -> Resistor_SMD:R_0805_2012Metric_Pad1.20x1.40mm_HandSolder
- SW1: value PP_BOOT -> BUTTON
Other:
- note added: "BOOT"
- moved on the sheet: C5, R1, SW1
