File: STLink.kicad_sch (KiCad schematic)
At the start: 42 parts, among them J2 JST, J3 MALE, J4 FEMALE, Q1 BC847, SW1 STLINK_BOOT, U1 STM32F103CBTx, U12 LP5907MFX-3.3, U5 SRV05-4, U6 SRV05-4, Y1 8M

Commit message: Consolidate BOM
Parts:
- D20: value RED -> ORANGE
- R12, R13, R14: value 220E -> 330E
- R8: value 1K5 -> 2K
- SW1: value STLINK_BOOT -> BUTTON
Other:
- note added: "BOOT"
