File: USBHS_FTDI.kicad_sch (KiCad schematic)
At the start: 56 parts, among them J13 FTDI, J14 UART1, J15 UART2, SW7 SW_DIP_x04, U12 LP5907MFX-3.3, U15 FT2232HL, U17 93LC66B, U6 SRV05-4, Y1 12MHz

Commit message: Consolidate BOM
Parts:
- D1: value UART 2 RX -> BLUE
- D1: value PWR -> ORANGE
- D1: value UART 2 TX -> BLUE
- D1: value UART 1 RX -> BLUE
- D1: value UART 1 TX -> BLUE
- FB2: value FBVPLL -> 600E-500mA
- J14: value UART1 -> UART
- J15: value UART2 -> UART
- R13: value 4K7 -> 5.1K
